File: first schematic.brd (EAGLE design)
At the start: 44.4 x 64.4 mm, 13 parts, among them IC1 ATMEGA328P, U1 ADXL362

Commit message: Add files via upload
Parts:
- removed B1: 3V, One_Dimensional_Pong:CR2450
- removed RESETSW: (no value), adafruit:BTN_CK_KSS
- added S1: EVP-BFAC1A000, EVP-BFAC1A000:EVPBFAC1A000
- added U$1, U$2, U$3: FIDUCIAL, adafruit:FIDUCIAL_1MM
- added U$4: CR2032, cr2032:CR2032
- moved U1 18.2 mm to (12.7, 17.8)
- moved J1 5.08 mm to (19.1, 59.7)
Connections:
- net GRND: now also S1.A2, U$4.GRND; no longer B1.GND, RESETSW.P$1
- net N$7: now also S1.A1; no longer RESETSW.P$2
- net VCC: now also U$4.VCC, U$4.VCC2; no longer B1.1, B1.2
Routing:
- net GRND: track 155.7 -> 184.2 mm, vias 6 -> 8
- net N$6: track 35.2 -> 54.7 mm, vias 0 -> 4
- net N$3: track 29.6 -> 44.6 mm, vias 0 -> 4
- net VCC: track 144.8 -> 130.0 mm, vias 1 -> 6
- net N$7: track 83.5 -> 78.5 mm, vias 1 -> 6
- net N$5: track 41.7 -> 46.4 mm, vias 2 -> 4
- net AREFTOCAP: track 25.7 -> 30.0 mm, vias 2 -> 4
- net N$10: track 29.4 -> 32.1 mm, vias 1 -> 0
- net N$8: track 31.0 -> 33.6 mm, vias 0 -> 2
- net N$2: track 26.2 -> 28.0 mm, vias 0 -> 2
- net N$9: track 28.9 -> 29.9 mm, vias 1 -> 0
Other:
- board text added: "11/12/2020"
- board text added: "Joshua Proulx"
- board text added: "Pedometer"
- board text added: "Rev 2"
- board text added: "https://github.com/jproulx1/388-Pedometer"
